File: 2019/KiCad_Badge/SMD/001_Template/001.kicad_pcb (KiCad board)
At the start: 2 copper layers, 0 parts

Commit message: Some minor updates 26-03-2019
Parts:
- added BT1: Battery_Cell, Battery:BatteryHolder_MPD_BC2003_1x2032, B.Cu at (165.7, 92.7)
- added C1: 10uF, Capacitor_SMD:C_1206_3216Metric, F.Cu at (158.1, 94.6)
- added D1: LED, LED_SMD:LED_1206_3216Metric_Pad1.42x1.75mm_HandSolder, F.Cu at (159.4, 87.6)
- added D2: LED, LED_SMD:LED_1206_3216Metric_Pad1.42x1.75mm_HandSolder, F.Cu at (174.6, 87.6)
- added R1: 1k, Resistor_SMD:R_1206_3216Metric_Pad1.42x1.75mm_HandSolder, F.Cu at (181.6, 87.6)
- added R2: 10k, Resistor_SMD:R_1206_3216Metric_Pad1.42x1.75mm_HandSolder, F.Cu at (176.5, 94.6)
- added R3: 1k, Resistor_SMD:R_1206_3216Metric_Pad1.42x1.75mm_HandSolder, F.Cu at (151.1, 87.6)
- added R4: 1k, Resistor_SMD:R_1206_3216Metric_Pad1.42x1.75mm_HandSolder, F.Cu at (166.4, 100.3)
- added U1: LM555, Package_SO:SOIC-8_3.9x4.9mm_P1.27mm, F.Cu at (166.0, 94.6)
