File: 2019/KiCad_Badge/SMD/001_Template/001.sch (KiCad schematic (older format))
At the start: 9 parts, among them U1 LM555

Commit message: Some minor updates 26-03-2019
Parts:
- BT1: footprint (none) -> Battery:BatteryHolder_MPD_BC2003_1x2032
- C1: footprint (none) -> Capacitor_SMD:C_1206_3216Metric
- D1, D2: footprint (none) -> LED_SMD:LED_1206_3216Metric_Pad1.42x1.75mm_HandSolder
- R1, R2, R3, R4: footprint (none) -> Resistor_SMD:R_1206_3216Metric_Pad1.42x1.75mm_HandSolder
- U1: footprint (none) -> Package_SO:SOIC-8_3.9x4.9mm_P1.27mm
Changed lines of the file:
@@
 F 0 "R3" H 7059 3596 50  0000 L CNN
 F 1 "1k" H 7059 3505 50  0000 L CNN
-F 2 "" H 7000 3550 50  0001 C CNN
+F 2 "Resistor_SMD:R_1206_3216Metric_Pad1.42x1.75mm_HandSolder" H 7000 3550 50  0001 C CNN
 F 3 "~" H 7000 3550 50  0001 C CNN
 	1    7000 3550
@@
 F 0 "R4" H 7059 4596 50  0000 L CNN
 F 1 "1k" H 7059 4505 50  0000 L CNN
-F 2 "" H 7000 4550 50  0001 C CNN
+F 2 "Resistor_SMD:R_1206_3216Metric_Pad1.42x1.75mm_HandSolder" H 7000 4550 50  0001 C CNN
 F 3 "~" H 7000 4550 50  0001 C CNN
 	1    7000 4550
@@
 F 0 "R2" H 4809 3696 50  0000 L CNN
 F 1 "10k" H 4809 3605 50  0000 L CNN
-F 2 "" H 4750 3650 50  0001 C CNN
+F 2 "Resistor_SMD:R_1206_3216Metric_Pad1.42x1.75mm_HandSolder" H 4750 3650 50  0001 C CNN
 F 3 "~" H 4750 3650 50  0001 C CNN
 	1    4750 3650
@@
 F 0 "R1" H 4809 3371 50  0000 L CNN
 F 1 "1k" H 4809 3280 50  0000 L CNN
-F 2 "" H 4750 3325 50  0001 C CNN
+F 2 "Resistor_SMD:R_1206_3216Metric_Pad1.42x1.75mm_HandSolder" H 4750 3325 50  0001 C CNN
 F 3 "~" H 4750 3325 50  0001 C CNN
 	1    4750 3325
@@
 F 0 "D1" V 7039 3733 50  0000 R CNN
 F 1 "LED" V 6948 3733 50  0000 R CNN
-F 2 "" H 7000 3850 50  0001 C CNN
+F 2 "LED_SMD:LED_1206_3216Metric_Pad1.42x1.75mm_HandSolder" H 7000 3850 50  0001 C CNN
 F 3 "~" H 7000 3850 50  0001 C CNN
 	1    7000 3850
@@
 F 0 "D2" V 7039 4133 50  0000 R CNN
 F 1 "LED" V 6948 4133 50  0000 R CNN
-F 2 "" H 7000 4250 50  0001 C CNN
+F 2 "LED_SMD:LED_1206_3216Metric_Pad1.42x1.75mm_HandSolder" H 7000 4250 50  0001 C CNN
 F 3 "~" H 7000 4250 50  0001 C CNN
 	1    7000 4250
@@
 F 0 "C1" H 4925 4075 50  0000 R CNN
 F 1 "10uF" H 5150 4250 50  0000 R CNN
-F 2 "" H 4750 4150 50  0001 C CNN
+F 2 "Capacitor_SMD:C_1206_3216Metric" H 4750 4150 50  0001 C CNN
 F 3 "~" H 4750 4150 50  0001 C CNN
 	1    4750 4150
@@
 F 0 "U1" H 5375 4650 50  0000 C CNN
 F 1 "LM555" H 5875 4650 50  0000 C CNN
-F 2 "" H 5650 4250 50  0001 C CNN
+F 2 "Package_SO:SOIC-8_3.9x4.9mm_P1.27mm" H 5650 4250 50  0001 C CNN
 F 3 "http://www.ti.com/lit/ds/symlink/lm555.pdf" H 5650 4250 50  0001 C CNN
 	1    5650 4250
@@
 F 0 "BT1" H 8818 3771 50  0000 L CNN
 F 1 "Battery_Cell" H 8818 3680 50  0000 L CNN
-F 2 "" V 8700 3735 50  0001 C CNN
+F 2 "Battery:BatteryHolder_MPD_BC2003_1x2032" V 8700 3735 50  0001 C CNN
 F 3 "~" V 8700 3735 50  0001 C CNN
 	1    8700 3675
