File: KiCad_Badge/SMD/001_Template/001.kicad_pcb (KiCad board)
At the start: 2 copper layers, 9 parts, among them U1 LM555

Commit message: Updates
Parts:
- removed BT1: Battery_Cell, Battery:BatteryHolder_MPD_BC2003_1x2032
- removed C1: 10uF, Capacitor_SMD:C_1206_3216Metric
- removed D1, D2: LED, LED_SMD:LED_1206_3216Metric_Pad1.42x1.75mm_HandSolder
- removed R1, R3, R4: 1k, Resistor_SMD:R_1206_3216Metric_Pad1.42x1.75mm_HandSolder
- removed R2: 10k, Resistor_SMD:R_1206_3216Metric_Pad1.42x1.75mm_HandSolder
- removed U1: LM555, Package_SO:SOIC-8_3.9x4.9mm_P1.27mm

Commit message: Updates
Parts:
- added BT1: Battery_Cell, Battery:BatteryHolder_MPD_BC2003_1x2032, F.Cu at (149.2, 95.2)
- added C1: 10uF, Capacitor_SMD:C_1206_3216Metric, F.Cu at (172.0, 99.4)
- added D1: LED, LED_SMD:LED_1206_3216Metric_Pad1.42x1.75mm_HandSolder, F.Cu at (166.2, 92.6)
- added D2: LED, LED_SMD:LED_1206_3216Metric_Pad1.42x1.75mm_HandSolder, F.Cu at (166.2, 96.0)
- added R1: 1k, Resistor_SMD:R_1206_3216Metric_Pad1.42x1.75mm_HandSolder, F.Cu at (172.2, 92.6)
- added R2: 10k, Resistor_SMD:R_1206_3216Metric_Pad1.42x1.75mm_HandSolder, F.Cu at (166.2, 99.4)
- added R3: 1k, Resistor_SMD:R_1206_3216Metric_Pad1.42x1.75mm_HandSolder, F.Cu at (172.2, 95.9)
- added R4: 1k, Resistor_SMD:R_1206_3216Metric_Pad1.42x1.75mm_HandSolder, F.Cu at (166.2, 102.6)
- added U1: LM555, Package_SO:SOIC-8_3.9x4.9mm_P1.27mm, F.Cu at (167.5, 87.7)
Other:
- board outline added: 95.8 x 87.2 mm
