File: KiCad_Badge/SMD/001_Template/001.sch (KiCad schematic (older format))
At the start: 9 parts, among them U1 LM555

Commit message: Minor updates
Parts:
- BT1: symbol Device:Battery_Cell -> 001-rescue:Battery_Cell-Device
- C1: symbol Device:C_Small -> 001-rescue:C_Small-Device
- D1, D2: symbol Device:LED -> 001-rescue:LED-Device
- R1, R2, R3, R4: symbol Device:R_Small -> 001-rescue:R_Small-Device
- U1: symbol Timer:LM555 -> 001-rescue:LM555-Timer
Changed lines of the file:
@@
 $EndBitmap
 $Comp
-L Device:R_Small R3
+L 001-rescue:R_Small-Device R3
 U 1 1 5CB4F2EF
 P 7000 3550
@@
 $EndComp
 $Comp
-L Device:R_Small R4
+L 001-rescue:R_Small-Device R4
 U 1 1 5CB50108
 P 7000 4550
@@
 $EndComp
 $Comp
-L Device:R_Small R2
+L 001-rescue:R_Small-Device R2
 U 1 1 5CB50538
 P 4750 3650
@@
 $EndComp
 $Comp
-L Device:R_Small R1
+L 001-rescue:R_Small-Device R1
 U 1 1 5CB50B08
 P 4750 3325
@@
 $EndComp
 $Comp
-L Device:LED D1
+L 001-rescue:LED-Device D1
 U 1 1 5CB5169F
 P 7000 3850
@@
 $EndComp
 $Comp
-L Device:LED D2
+L 001-rescue:LED-Device D2
 U 1 1 5CB5226B
 P 7000 4250
@@
 $EndComp
 $Comp
-L Device:C_Small C1
+L 001-rescue:C_Small-Device C1
 U 1 1 5CB532FA
 P 4750 4150
@@
 $EndComp
 $Comp
-L Timer:LM555 U1
+L 001-rescue:LM555-Timer U1
 U 1 1 5CB43957
 P 5650 4250
@@
 	4750 3150 4750 3225
 $Comp
-L Device:Battery_Cell BT1
+L 001-rescue:Battery_Cell-Device BT1
 U 1 1 5CB57B92
 P 8700 3675

Commit message: Updates
Parts:
- BT1: symbol 001-rescue:Battery_Cell-Device -> 001-rescue:Battery_Cell-Device-001-rescue
- C1: symbol 001-rescue:C_Small-Device -> 001-rescue:C_Small-Device-001-rescue
- D1, D2: symbol 001-rescue:LED-Device -> 001-rescue:LED-Device-001-rescue
- R1, R2, R3, R4: symbol 001-rescue:R_Small-Device -> 001-rescue:R_Small-Device-001-rescue
- U1: symbol 001-rescue:LM555-Timer -> 001-rescue:LM555-Timer-001-rescue
Changed lines of the file:
@@
 $EndBitmap
 $Comp
-L 001-rescue:R_Small-Device R3
+L 001-rescue:R_Small-Device-001-rescue R3
 U 1 1 5CB4F2EF
 P 7000 3550
@@
 $EndComp
 $Comp
-L 001-rescue:R_Small-Device R4
+L 001-rescue:R_Small-Device-001-rescue R4
 U 1 1 5CB50108
 P 7000 4550
@@
 $EndComp
 $Comp
-L 001-rescue:R_Small-Device R2
+L 001-rescue:R_Small-Device-001-rescue R2
 U 1 1 5CB50538
 P 4750 3650
@@
 $EndComp
 $Comp
-L 001-rescue:R_Small-Device R1
+L 001-rescue:R_Small-Device-001-rescue R1
 U 1 1 5CB50B08
 P 4750 3325
@@
 $EndComp
 $Comp
-L 001-rescue:LED-Device D1
+L 001-rescue:LED-Device-001-rescue D1
 U 1 1 5CB5169F
 P 7000 3850
@@
 $EndComp
 $Comp
-L 001-rescue:LED-Device D2
+L 001-rescue:LED-Device-001-rescue D2
 U 1 1 5CB5226B
 P 7000 4250
@@
 $EndComp
 $Comp
-L 001-rescue:C_Small-Device C1
+L 001-rescue:C_Small-Device-001-rescue C1
 U 1 1 5CB532FA
 P 4750 4150
@@
 $EndComp
 $Comp
-L 001-rescue:LM555-Timer U1
+L 001-rescue:LM555-Timer-001-rescue U1
 U 1 1 5CB43957
 P 5650 4250
@@
 	4750 3150 4750 3225
 $Comp
-L 001-rescue:Battery_Cell-Device BT1
+L 001-rescue:Battery_Cell-Device-001-rescue BT1
 U 1 1 5CB57B92
 P 8700 3675
